Commit message: [feat]: enable lidar sensor, but need to downsample 10x

File: realsense_gazebo_plugin/urdf/realsense-RS200.macro.xacro (robot description, xacro)
@@ -23,17 +23,16 @@
         <collision>
             <geometry>
-                <box size="0.0078 0.130 0.0192"/>
+                <box size="0.001 0.001 0.001"/>
             </geometry>
         </collision>
         <inertial>
-            <!-- <mass value="0.0615752"/> -->
-            <mass value="0.00000001"/>
+            <mass value="0.0001"/>
             <origin rpy="0 0 0" xyz="0 0 0"/>
-            <inertia ixx="9.108e-05"
+            <inertia ixx="0.00001"
                      ixy="0"
                      ixz="0"
-                     iyy="2.51e-06"
+                     iyy="0.00001"
                      iyz="0"
-                     izz="8.931e-05"
+                     izz="0.00001"
             />
         </inertial>
@@ -93,6 +92,6 @@
         <!--<slip1>0</slip1>
         <slip2>0</slip2>-->
-        <kp>1e+13</kp>
-        <kd>1</kd>
+        <!-- <kp>1e+13</kp>
+        <kd>1</kd> -->
         <!--<max_vel>0.01</max_vel>
         <min_depth>0</min_depth>-->

File: realsense_gazebo_plugin/urdf/rs200_simulation.xacro (robot description, xacro)
@@ -11,5 +11,5 @@
     <!-- <xacro:realsense-rs200 prefix="" parent="world"> -->
     <xacro:realsense-rs200 prefix="">
-        <origin xyz="0 0 1.0" rpy="0 0 0" />
+        <origin xyz="0 0 0" rpy="0 0 0" />
     </xacro:realsense-rs200>
 </robot>

File: unitree_ros/robots/go2_description/xacro/robot_with_sensor.xacro (robot description, xacro)
@@ -1,12 +1,19 @@
 <?xml version="1.0"?>
 <robot name="combined_robot" xmlns:xacro="http://ros.org/wiki/xacro">
-  <!-- Include the two robots -->
+  <!-- Include robot and sensor -->
   <xacro:include filename="$(find go2_description)/xacro/robot.xacro"/>
   <xacro:include filename="$(find realsense_gazebo_plugin)/urdf/rs200_simulation.xacro"/>
-  <!-- Define the fixed joint to link the robots rigidly -->
-  <joint name="fixed_joint_between_robots" type="fixed">
+  <xacro:include filename="$(find livox_laser_simulation)/urdf/livox_mid360.xacro"/>
+  <!-- <xacro:include filename="$(find livox_laser_simulation_new)/models/sensors_only/model.xacro"/> -->
+  <!-- Define the fixed joint to link the robot and sensor -->
+  <joint name="fixed_joint_between_robot_and_rgbd" type="fixed">
     <parent link="base"/>
     <child link="rs200_camera"/>
-    <origin xyz="1 1 1" rpy="0 0 0"/>
+    <origin xyz="0.35 0 0.1" rpy="0 0 0"/>
+  </joint>
+  <joint name="fixed_joint_between_robot_and_lidar" type="fixed">
+    <parent link="base"/>
+    <child link="livox_base"/>
+    <origin xyz="0.35 0 0.2" rpy="0 0 0"/>
   </joint>
 </robot>
