Commit message: [feat]: add ugv car

File: livox_laser_simulation/urdf/livox_mid360.xacro (robot description, xacro)
@@ -6,5 +6,5 @@
   <xacro:property name="ros_topic" value="scan"/>
   <xacro:property name="samples" value="24000"/>
-  <xacro:property name="downsample" value="10"/>
+  <xacro:property name="downsample" value="4"/>
   <xacro:macro name="null_inertial">
     <inertial>

File: realsense_gazebo_plugin/urdf/realsense-RS200.macro.xacro (robot description, xacro)
@@ -102,5 +102,5 @@
             <image>
                 <width>640</width>
-                <height>480</height>
+                <height>360</height>
                 <format>RGB_INT8</format>
             </image>
@@ -112,10 +112,11 @@
                 <type>gaussian</type>
                 <mean>0.0</mean>
-                <stddev>0.007</stddev>
+                <!-- <stddev>0.007</stddev> -->
+                <stddev>0.0</stddev>
             </noise>
             </camera>
             <always_on>1</always_on>
-            <update_rate>60</update_rate>
-            <visualize>1</visualize>
+            <update_rate>30</update_rate>
+            <visualize>0</visualize>
         </sensor>
         <sensor name="${prefix}ired1" type="camera">
@@ -125,5 +126,5 @@
             <image>
                 <width>640</width>
-                <height>480</height>
+                <height>360</height>
                 <format>L_INT8</format>
             </image>
@@ -135,9 +136,10 @@
                 <type>gaussian</type>
                 <mean>0.0</mean>
-                <stddev>0.05</stddev>
+                <!-- <stddev>0.05</stddev> -->
+                <stddev>0.0</stddev>
             </noise>
             </camera>
-            <always_on>1</always_on>
-            <update_rate>60</update_rate>
+            <always_on>0</always_on>
+            <update_rate>30</update_rate>
             <visualize>0</visualize>
         </sensor>
@@ -148,5 +150,5 @@
             <image>
                 <width>640</width>
-                <height>480</height>
+                <height>360</height>
                 <format>L_INT8</format>
             </image>
@@ -158,9 +160,10 @@
                 <type>gaussian</type>
                 <mean>0.0</mean>
-                <stddev>0.05</stddev>
+                <!-- <stddev>0.05</stddev> -->
+                <stddev>0.0</stddev>
             </noise>
             </camera>
-            <always_on>1</always_on>
-            <update_rate>60</update_rate>
+            <always_on>0</always_on>
+            <update_rate>30</update_rate>
             <visualize>0</visualize>
         </sensor>
@@ -171,5 +174,5 @@
             <image>
                     <width>640</width>
-                    <height>480</height>
+                    <height>360</height>
             </image>
             <clip>
@@ -180,9 +183,10 @@
                     <type>gaussian</type>
                     <mean>0.0</mean>
-                    <stddev>0.100</stddev>
+                    <!-- <stddev>0.100</stddev> -->
+                    <stddev>0.0</stddev>
             </noise>
             </camera>
             <always_on>1</always_on>
-            <update_rate>60</update_rate>
+            <update_rate>30</update_rate>
             <visualize>0</visualize>
         </sensor>
